Commit message: .

File: assets/robot.urdf (robot description, URDF)
Before this commit: robot folderv2, 27 links, 26 joints
Joints:
- joint base_yaw: type revolute -> fixed

Commit message: change positions

File: assets/robot.urdf (robot description, URDF)
Before this commit: robot folderv2, 27 links, 26 joints
Links:
- added link world
Joints:
- added joint fixed: type fixed, parent world, child base_new, origin xyz=0 0 0 rpy=-1.5708 0 0
